File: Schematic/KiCad/HM-Sensor.kicad_pcb (KiCad board)
At the start: 2 copper layers, 62 x 62 mm, 37 parts, among them J1 BAT+, J2 BAT-, J3 Serial, J4 GS2, J5 ISP, J6 VCC-Src, J7 I2C, J8 A0-A7, SW1 SW_Push, U1 MAX1724+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

Commit message: pcb routing complete
Parts:
- moved C4 0.65 mm to (110.1, 114.3)
- moved C7 0.64 mm to (111.9, 114.3)
- moved C1 0.50 mm to (111.8, 97.5)
- moved C5 0.50 mm to (113.7, 97.5)
Routing:
- net +3V3: track 76.1 -> 136.4 mm, vias 2 -> 8
- net GND: track 135.5 -> 179.7 mm, vias 0 -> 4
- net /SDA: track 0.00 -> 42.4 mm, vias 0 -> 3
- net /SCL: track 0.00 -> 38.3 mm, vias 0 -> 2
- net /A0: track 0.00 -> 38.1 mm, vias 0 -> 2
- net /A3: track 0.00 -> 36.7 mm, vias 0 -> 1
- net /A2: track 0.00 -> 36.7 mm, vias 0 -> 1
- net /B2: track 0.00 -> 34.4 mm, vias 0 -> 2
- net /B1: track 0.00 -> 33.6 mm, vias 0 -> 2
- net /A6: track 0.00 -> 32.4 mm, vias 0 -> 2
- net /A7: track 0.00 -> 31.2 mm, vias 0 -> 2
- net /MISO: track 21.1 -> 51.7 mm, vias 1 -> 2
- net /SCK: track 20.8 -> 44.0 mm, vias 1 -> 3
- net /MOSI: track 12.2 -> 32.5 mm, vias 1 -> 3
- net /U-Sens: track 27.1 -> 34.0 mm
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- added copper zone on B.Cu, net GND
- added copper zone on F.Cu, net GND
Other:
- net class Default: clearance 0.2 -> 0.205
- net class Power: clearance 0.2 -> 0.205
- net class Thin: clearance 0.2 -> 0.205
- rule pad_to_mask_clearance: 0.2 -> 0.15
- rule trace_clearance: 0.2 -> 0.205
- rule trace_min: 0.2 -> 0.21

Commit message: went to production
Parts:
- moved C7 0.80 mm to (111.1, 114.3)
- moved C4 0.60 mm to (109.5, 114.3)
Connections:
- REF1 pad 1: (no net) -> /U-BAT
- REF1 pad 2: (no net) -> GND
Routing:
- net GND: track 179.7 -> 210.4 mm, vias 4 -> 5
- net /U-BAT: track 28.4 -> 56.7 mm
- net +3V3: track 136.4 -> 131.7 mm
- net /SCK: track 44.0 -> 47.1 mm
- net /MISO: track 51.7 -> 53.8 mm
- net /D2: track 26.8 -> 28.7 mm
- net Net-(U3-Pad7): track 0.00 -> 1.75 mm
- net /U-Sens: track 34.0 -> 32.7 mm
- net /A7: track 31.2 -> 32.4 mm
- net /MOSI: track 32.5 -> 33.6 mm
- net /A1: track 14.2 -> 13.2 mm
- net /SDA: track 42.4 -> 43.1 mm
Other:
- outline, holes or cut-outs redrawn
- board text added: "HM-Sensor Rev 2.0a"

Commit message: better ground layout
Parts:
- added REF**: 0,3mm-VIA, MyLibs:VIA-0,3mm, F.Cu at (122.3, 82.2)
- added REF**: 0,3mm-VIA, MyLibs:VIA-0,3mm, F.Cu at (120.4, 84.6)
- added REF**: 0,3mm-VIA, MyLibs:VIA-0,3mm, F.Cu at (116.9, 90.1)
- added REF**: 0,3mm-VIA, MyLibs:VIA-0,3mm, F.Cu at (116.1, 92.4)
- added REF**: 0,3mm-VIA, MyLibs:VIA-0,3mm, F.Cu at (112.5, 111.7)
- added REF**: 0,3mm-VIA, MyLibs:VIA-0,3mm, F.Cu at (113.5, 115.6)
- added REF**: 0,3mm-VIA, MyLibs:VIA-0,3mm, F.Cu at (108.6, 117.9)
- added REF**: 0,3mm-VIA, MyLibs:VIA-0,3mm, F.Cu at (115.3, 122.3)
- added REF**: 0,3mm-VIA, MyLibs:VIA-0,3mm, F.Cu at (115.3, 124.2)
Changed lines of the file:
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@@
 (kicad_pcb (version 4) (host pcbnew 4.0.6)
   (general
-    (links 97)
+    (links 106)
     (no_connects 0)
     (area 59.650001 78.893999 165.047859 153.200001)
     (thickness 1.6)
     (drawings 29)
-    (tracks 588)
+    (tracks 592)
     (zones 0)
-    (modules 37)
+    (modules 46)
     (nets 39)
   )
@@
   )
   (setup
-    (last_trace_width 0.25)
+    (last_trace_width 0.4)
     (user_trace_width 0.25)
     (user_trace_width 0.4)
@@
     (mod_text_size 0.8 0.8)
     (mod_text_width 0.15)
-    (pad_size 2.4 2.4)
-    (pad_drill 2.4)
+    (pad_size 0.5 0.5)
+    (pad_drill 0.3)
     (pad_to_mask_clearance 0.15)
     (solder_mask_min_width 0.15)
@@
     (pcbplotparams
       (layerselection 0x010f0_80000001)
-      (usegerberextensions true)
+      (usegerberextensions false)
       (excludeedgelayer true)
       (linewidth 0.100000)
@@
       (padsonsilk false)
       (subtractmaskfromsilk false)
-      (outputformat 1)
+      (outputformat 4)
       (mirror false)
-      (drillshape 0)
+      (drillshape 2)
       (scaleselection 1)
       (outputdirectory ""))
@@
     (add_net /XTAL2)
   )
+  (module MyLibs:VIA-0,3mm (layer F.Cu)
+    (at 122.3 82.2)
+    (fp_text reference REF** (at 0 1.2) (layer F.SilkS) hide
+      (effects (font (size 1 1) (thickness 0.15)))
+    )
+    (fp_text value 0,3mm-VIA (at 0 -1.1) (layer F.Fab) hide
+      (effects (font (size 1 1) (thickness 0.15)))
+    )
+    (pad 1 thru_hole circle (at 0 0) (size 0.5 0.5) (drill 0.3) (layers *.Cu)
+      (net 3 GND) (zone_connect 2))
+  )
+  (module MyLibs:VIA-0,3mm (layer F.Cu)
+    (at 120.4 84.6)
+    (fp_text reference REF** (at 0 1.2) (layer F.SilkS) hide
+      (effects (font (size 1 1) (thickness 0.15)))
+    )
+    (fp_text value 0,3mm-VIA (at 0 -1.1) (layer F.Fab) hide
+      (effects (font (size 1 1) (thickness 0.15)))
+    )
+    (pad 1 thru_hole circle (at 0 0) (size 0.5 0.5) (drill 0.3) (layers *.Cu)
+      (net 3 GND) (zone_connect 2))
+  )
+  (module MyLibs:VIA-0,3mm (layer F.Cu)
+    (at 116.9 90.1)
+    (fp_text reference REF** (at 0 1.2) (layer F.SilkS) hide
+      (effects (font (size 1 1) (thickness 0.15)))
+    )
+    (fp_text value 0,3mm-VIA (at 0 -1.1) (layer F.Fab) hide
+      (effects (font (size 1 1) (thickness 0.15)))
+    )
+    (pad 1 thru_hole circle (at 0 0) (size 0.5 0.5) (drill 0.3) (layers *.Cu)
+      (net 3 GND) (zone_connect 2))
+  )
+  (module MyLibs:VIA-0,3mm (layer F.Cu)
+    (at 116.1 92.4)
+    (fp_text reference REF** (at 0 1.2) (layer F.SilkS) hide
+      (effects (font (size 1 1) (thickness 0.15)))
+    )
+    (fp_text value 0,3mm-VIA (at 0 -1.1) (layer F.Fab) hide
+      (effects (font (size 1 1) (thickness 0.15)))
+    )
+    (pad 1 thru_hole circle (at 0 0) (size 0.5 0.5) (drill 0.3) (layers *.Cu)
+      (net 3 GND) (zone_connect 2))
+  )
+  (module MyLibs:VIA-0,3mm (layer F.Cu)
+    (at 112.5 111.7)
+    (fp_text reference REF** (at 0 1.2) (layer F.SilkS) hide
+      (effects (font (size 1 1) (thickness 0.15)))
+    )
+    (fp_text value 0,3mm-VIA (at 0 -1.1) (layer F.Fab) hide
+      (effects (font (size 1 1) (thickness 0.15)))
+    )
+    (pad 1 thru_hole circle (at 0 0) (size 0.5 0.5) (drill 0.3) (layers *.Cu)
+      (net 3 GND) (zone_connect 2))
+  )
+  (module MyLibs:VIA-0,3mm (layer F.Cu)
+    (at 113.5 115.6)
+    (fp_text reference REF** (at 0 1.2) (layer F.SilkS) hide
+      (effects (font (size 1 1) (thickness 0.15)))
+    )
+    (fp_text value 0,3mm-VIA (at 0 -1.1) (layer F.Fab) hide
+      (effects (font (size 1 1) (thickness 0.15)))
+    )
+    (pad 1 thru_hole circle (at 0 0) (size 0.5 0.5) (drill 0.3) (layers *.Cu)
+      (net 3 GND) (zone_connect 2))
+  )
+  (module MyLibs:VIA-0,3mm (layer F.Cu)
+    (at 108.6 117.9)
+    (fp_text reference REF** (at 0 1.2) (layer F.SilkS) hide
+      (effects (font (size 1 1) (thickness 0.15)))
+    )
+    (fp_text value 0,3mm-VIA (at 0 -1.1) (layer F.Fab) hide
+      (effects (font (size 1 1) (thickness 0.15)))
+    )
+    (pad 1 thru_hole circle (at 0 0) (size 0.5 0.5) (drill 0.3) (layers *.Cu)
+      (net 3 GND) (zone_connect 2))
+  )
+  (module MyLibs:VIA-0,3mm (layer F.Cu)
+    (at 115.3 122.3)
+    (fp_text reference REF** (at 0 1.2) (layer F.SilkS) hide
+      (effects (font (size 1 1) (thickness 0.15)))
+    )
+    (fp_text value 0,3mm-VIA (at 0 -1.1) (layer F.Fab) hide
+      (effects (font (size 1 1) (thickness 0.15)))
+    )
+    (pad 1 thru_hole circle (at 0 0) (size 0.5 0.5) (drill 0.3) (layers *.Cu)
+      (net 3 GND) (zone_connect 2))
+  )
   (module Pin_Headers:Pin_Header_Straight_1x04_Pitch2.54mm (layer F.Cu)
     (at 99.949 110.744)
@@
       (net 3 GND))
     (pad 3 smd rect (at 1 1.4 90) (size 0.4 0.6) (layers F.Cu F.Mask))
+  )
+  (module MyLibs:VIA-0,3mm (layer F.Cu)
+    (at 115.3 124.2)
+    (fp_text reference REF** (at 0 1.2) (layer F.SilkS) hide
+      (effects (font (size 1 1) (thickness 0.15)))
+    )
+    (fp_text value 0,3mm-VIA (at 0 -1.1) (layer F.Fab) hide
+      (effects (font (size 1 1) (thickness 0.15)))
+    )
+    (pad 1 thru_hole circle (at 0 0) (size 0.5 0.5) (drill 0.3) (layers *.Cu)
+      (net 3 GND) (zone_connect 2))
   )
   (gr_text "HM-Sensor Rev 2.0a" (at 158.58 108.84 270) (layer B.Cu)
@@
   (segment (start 107.881099 132.694501) (end 106.902999 131.716401) (width 0.4) (layer B.Cu) (net 27))
   (via (at 104.504112 110.923786) (size 0.7) (drill 0.5) (layers F.Cu B.Cu) (net 27))
-  (segment (start 119.485 126.897) (end 119.104 126.897) (width 0.4) (layer F.Cu) (net 28) (status 30))
-  (segment (start 119.104 126.897) (end 115.651 123.444) (width 0.4) (layer F.Cu) (net 28) (status 10))
-  (segment (start 115.651 123.444) (end 109.4105 123.444) (width 0.4) (layer F.Cu) (net 28))
-  (segment (start 109.4105 123.444) (end 106.9975 121.031) (width 0.4) (layer F.Cu) (net 28))
-  (segment (start 106.9975 121.031) (end 106.9975 116.9035) (width 0.4) (layer F.Cu) (net 28))
+  (segment (start 117.942 125.652078) (end 115.685921 123.395999) (width 0.4) (layer F.Cu) (net 28))
+  (segment (start 106.9975 121.031) (end 106.9975 117.398474) (width 0.4) (layer F.Cu) (net 28))
+  (segment (start 106.9975 117.398474) (end 106.9975 116.9035) (width 0.4) (layer F.Cu) (net 28))
+  (segment (start 109.362499 123.395999) (end 106.9975 121.031) (width 0.4) (layer F.Cu) (net 28))
+  (segment (start 115.685921 123.395999) (end 109.362499 123.395999) (width 0.4) (layer F.Cu) (net 28))
+  (segment (start 117.942 125.735) (end 117.942 125.652078) (width 0.4) (layer F.Cu) (net 28))
+  (segment (start 119.104 126.897) (end 117.942 125.735) (width 0.4) (layer F.Cu) (net 28))
+  (segment (start 119.485 126.897) (end 119.104 126.897) (width 0.4) (layer F.Cu) (net 28))
   (segment (start 121.235 126.897) (end 119.485 126.897) (width 0.4) (layer F.Cu) (net 28) (status 30))
   (segment (start 106.9975 116.9035) (end 105.360012 115.266012) (width 0.4) (layer B.Cu) (net 28))
@@
   (segment (start 107.891 107.118) (end 105.182 107.118) (width 0.4) (layer F.Cu) (net 28) (status 10))
   (via (at 106.9975 116.9035) (size 0.7) (drill 0.5) (layers F.Cu B.Cu) (net 28))
+  (segment (start 113.823001 112.808499) (end 114.173 112.4585) (width 0.4) (layer B.Cu) (net 29))
+  (segment (start 112.294998 114.336502) (end 113.823001 112.808499) (width 0.4) (layer B.Cu) (net 29))
+  (segment (start 112.294998 122.38492) (end 112.294998 114.336502) (width 0.4) (layer B.Cu) (net 29))
+  (segment (start 116.084977 126.174899) (end 112.294998 122.38492) (width 0.4) (layer B.Cu) (net 29))
+  (segment (start 116.084977 131.350001) (end 116.084977 126.174899) (width 0.4) (layer B.Cu) (net 29))
+  (segment (start 115.734978 131.7) (end 116.084977 131.350001) (width 0.4) (layer B.Cu) (net 29))
   (segment (start 114.141 112.4265) (end 114.173 112.4585) (width 0.4) (layer F.Cu) (net 29))
   (segment (start 114.141 110.168) (end 114.141 112.4265) (width 0.4) (layer F.Cu) (net 29) (status 10))
-  (segment (start 112.294998 114.336502) (end 114.173 112.4585) (width 0.4) (layer B.Cu) (net 29))
-  (segment (start 116.084977 126.084977) (end 112.294998 122.294998) (width 0.4) (layer B.Cu) (net 29))
-  (segment (start 112.294998 122.294998) (end 112.294998 114.336502) (width 0.4) (layer B.Cu) (net 29))
-  (segment (start 116.084977 131.350001) (end 116.084977 126.084977) (width 0.4) (layer B.Cu) (net 29))
-  (segment (start 115.734978 131.7) (end 116.084977 131.350001) (width 0.4) (layer B.Cu) (net 29))
   (via (at 114.173 112.4585) (size 0.7) (drill 0.5) (layers F.Cu B.Cu) (net 29))
   (segment (start 114.465978 132.969) (end 115.734978 131.7) (width 0.4) (layer F.Cu) (net 29))
@@
   (zone (net 3) (net_name GND) (layer F.Cu) (hatch edge 0.508)
     (connect_pads (clearance 0.381))
-    (min_thickness 0.254)
-    (fill yes (arc_segments 16) (thermal_gap 0.508) (thermal_bridge_width 0.508))
+    (min_thickness 0.1524)
+    (fill yes (arc_segments 32) (thermal_gap 0.508) (thermal_bridge_width 0.508))
     (polygon
       (pts
@@
   (zone (net 3) (net_name GND) (layer B.Cu) (hatch edge 0.508)
     (connect_pads (clearance 0.381))
-    (min_thickness 0.254)
-    (fill yes (arc_segments 16) (thermal_gap 0.508) (thermal_bridge_width 0.508))
+    (min_thickness 0.1524)
+    (fill yes (arc_segments 32) (thermal_gap 0.508) (thermal_bridge_width 0.508))
     (polygon
       (pts
